File: kicad/template/template.kicad_sch (KiCad schematic)
At the start: 0 parts

Commit message: remove MRC branding
Other:
- company: BU Mars Rover Club Electrical Team -> Boston University College of Engineering
- title: ${MRC_TITLE} -> ${SCH_TITLE}
